Commit message: update xacro setup for the robot

File: stretch_description/urdf/stretch_laser_range_finder.xacro (robot description, xacro)
@@ -32,4 +32,10 @@
     </visual>
     <collision>
+      <origin rpy="-1.570796 1.570796 1.570796" xyz="-0.000750 0.000000 0.000000"/>
+      <geometry>
+        <box size="0.019500 0.069940 0.069940"/>
+      </geometry>
+    </collision>
+    <!--collision>
       <origin
         xyz="0 0 0"
@@ -39,5 +45,5 @@
           filename="package://stretch_description/meshes/laser.STL" />
       </geometry>
-    </collision>
+    </collision-->
   </link>
   <joint
